File: boards/cfxsx.kicad_pcb (KiCad board)
At the start: 4 copper layers, 29 x 61.6 mm, 22 parts, among them J1 M.2 NGFF

Commit message: Deploying to gh-pages from @ neg2led/cfxsx@5fded029270c65b2b62c4b467ed82b7d2456e2af 🚀
Parts:
- removed the REF** at (139.5, 116.0)
- added MP2: 2242, 11-My-Edits:MountingHole_NGFF_4.2mm_Pad_TopBottom, B.Cu at (150.0, 127.5)
- REF**: renamed from MP2; value 2242 -> mousebite; footprint 11-My-Edits:MountingHole_NGFF_4.2mm_Pad_TopBottom -> 10-My-Footprints:mousebite; moved to F.Cu
- moved REF** 21.1 mm to (139.5, 113.0)
- moved REF** 17.9 mm to (160.5, 113.0)
- moved REF** 3.00 mm to (139.5, 118.0)
- moved REF** 3.00 mm to (160.5, 115.0)
- moved REF** 3.00 mm to (139.5, 117.0)
- moved REF** 2.00 mm to (139.5, 115.0)
- moved REF** 2.00 mm to (139.5, 116.0)
- moved REF** 2.00 mm to (160.5, 116.0)
- moved REF** 1.00 mm to (160.5, 114.0)
- moved REF** 1.00 mm to (160.5, 117.0)
- moved REF** 1.00 mm to (160.5, 118.0)
- moved REF** 1.00 mm to (139.5, 114.0)
